File: PCB/PCB.kicad_pcb (KiCad board)
At the start: 2 copper layers, 62.5 x 66.7 mm, 10 parts, among them SW1 SW_Push, SW2 SW_Push, SW3 SW_Push, SW4 SW_Push, SW5 SW_Push, SW6 SW_Push, SW7 SW_Push, U1 XIAO-RP2040-DIP

Commit message: Add files via upload
Parts:
- removed D1, D2: SK6812MINI, LED_SMD:LED_SK6812MINI_PLCC4_3.5x3.5mm_P1.75mm
- added SW8: RotaryEncoder_Switch, Rotary_Encoder:RotaryEncoder_Alps_EC11E-Switch_Vertical_H20mm, F.Cu at (109.4, 98.0)
Connections:
- U1 pad 4: unconnected-(U1-GPIO29/ADC3/A3-Pad4) -> Net-(U1-GPIO29/ADC3/A3)
- U1 pad 6: unconnected-(U1-GPIO7/SCL-Pad6) -> Net-(U1-GPIO7/SCL)
- U1 pad 7: unconnected-(U1-GPIO0/TX-Pad7) -> Net-(U1-GPIO0/TX)
Routing:
- net +5V: track 60.7 -> 0.00 mm
- net Net-(U1-GPIO29/ADC3/A3): track 0.00 -> 50.4 mm
- net Net-(U1-GPIO7/SCL): track 0.00 -> 29.3 mm
- net Net-(U1-GPIO0/TX): track 0.00 -> 25.3 mm
- net Net-(U1-GPIO6/SDA): track 35.8 -> 48.2 mm
- net GND: track 156.8 -> 145.6 mm
- net Net-(D1-DOUT): track 7.14 -> 0.00 mm
- net Net-(U1-GPIO1/RX): track 25.2 -> 21.7 mm, vias 1 -> 0
