File: PCB/PCB.kicad_sch (KiCad schematic)
At the start: 10 parts, among them SW1 SW_Push, SW2 SW_Push, SW3 SW_Push, SW4 SW_Push, SW5 SW_Push, SW6 SW_Push, SW7 SW_Push, U1 XIAO-RP2040-DIP

Commit message: Add files via upload
Parts:
- removed D1, D2: SK6812MINI, LED_SMD:LED_SK6812MINI_PLCC4_3.5x3.5mm_P1.75mm, symbol LED:SK6812MINI
- added SW8: RotaryEncoder_Switch, Rotary_Encoder:RotaryEncoder_Alps_EC11E-Switch_Vertical_H20mm, symbol Device:RotaryEncoder_Switch
Connections:
- net GND: now also SW8.C
- net at U1.5 (GPIO6/SDA): now also SW8.A
- net at U1.4 (GPIO29/ADC3/A3): now also SW8.B
- net at U1.6 (GPIO7/SCL): now also SW8.S1
- net at U1.7 (GPIO0/TX): now also SW8.S2
